File: solder.kicad_pcb (KiCad board)
At the start: 2 copper layers, 5 parts

Commit message: PCB Draft 1
Parts:
- removed D2: LED, LED_THT:LED_D5.0mm
- removed R2: R, Resistor_THT:R_Axial_DIN0207_L6.3mm_D2.5mm_P7.62mm_Horizontal
- added G***: LOGO, LOGO, F.Cu at (136.4, 103.0)
- added Q1: NPN, Package_TO_SOT_THT:TO-92L_HandSolder, B.Cu at (156.0, 82.0)
- added RV1: R_Potentiometer, Potentiometer_THT:Potentiometer_Vishay_T73YP_Vertical, B.Cu at (115.0, 97.5)
- added RV2: R_Potentiometer, Potentiometer_THT:Potentiometer_Vishay_T73YP_Vertical, B.Cu at (117.5, 85.0)
- BT1: moved to B.Cu
- R1: value R -> R_Photo; footprint Resistor_THT:R_Axial_DIN0207_L6.3mm_D2.5mm_P7.62mm_Horizontal -> OptoDevice:R_LDR_5.1x4.3mm_P3.4mm_Vertical
- moved BT1 82.0 mm to (137.5, 99.0), turned to 180 degrees
- moved R1 74.8 mm to (155.6, 99.1), turned to 90 degrees
- moved D1 41.8 mm to (149.5, 69.0)
Connections:
- D1 pad 2: Net-(BT1-+) -> Net-(D1-A)
- R1 pad 1: Net-(D1-K) -> Net-(Q1-B)
Routing:
- net Net-(Q1-B): track 0.00 -> 64.0 mm, vias 0 -> 1
- net Net-(BT1-+): track 0.00 -> 58.2 mm
- net Net-(D1-K): track 0.00 -> 38.0 mm, vias 0 -> 1
- net Net-(BT1--): track 0.00 -> 32.7 mm, vias 0 -> 1
- net Net-(D1-A): track 0.00 -> 14.6 mm, vias 0 -> 1
Other:
- board outline added: 59.6 x 53.6 mm
- board text added: "obob"
