File: solder.kicad_pcb (KiCad board)
At the start: 2 copper layers, 59.6 x 53.6 mm, 7 parts, among them Q1 NPN

Commit message: add resistor
Parts:
- added R2: 5K1, Resistor_THT:R_Axial_DIN0207_L6.3mm_D2.5mm_P7.62mm_Horizontal, B.Cu at (141.7, 82.6)
Connections:
- RV1 pad 2: Net-(Q1-B) -> Net-(R2-Pad1)
Routing:
- net Net-(Q1-B): track 64.0 -> 27.2 mm
- net Net-(R2-Pad1): track 0.00 -> 29.3 mm

Commit message: update images and pcb
Parts:
- added R3: 5K1, Resistor_THT:R_Axial_DIN0207_L6.3mm_D2.5mm_P7.62mm_Horizontal, B.Cu at (151.6, 87.4)
- G***: moved to B.Cu
- moved G*** 29.7 mm to (143.3, 74.1), turned to 180 degrees
Connections:
- R2 pad 2: Net-(Q1-B) -> Net-(R2-Pad2)
Routing:
- net Net-(R2-Pad2): track 0.00 -> 7.33 mm
- net Net-(Q1-B): track 27.2 -> 29.7 mm
Other:
- board text added: "quack"
- board text removed: "obob"
