File: solder.kicad_pcb (KiCad board)
At the start: 2 copper layers, 59.6 x 53.6 mm, 9 parts, among them Q1 NPN

Commit message: update silkscreen
Parts:
- added G***: LOGO, LOGO, F.Cu at (122.0, 92.0)
- added G***: LOGO, LOGO, F.Cu at (143.9, 72.4)
- added G***: LOGO, LOGO, F.Cu at (143.9, 94.5)

Commit message: add production files
Parts:
- removed the G*** at (122.0, 92.0)
- removed the G*** at (143.9, 72.4)
- removed the G*** at (143.9, 94.5)
- added G***: LOGO, LOGO, F.Cu at (139.8, 70.7)
- added G***: LOGO, LOGO, F.Cu at (147.4, 85.4)
- added G***: LOGO, LOGO, F.Cu at (137.3, 99.2)
- added G***: LOGO, LOGO, F.Cu at (161.2, 75.0)
- added G***: LOGO, LOGO, F.Cu at (126.2, 86.1)
Other:
- board text added: "North Sydney Boys High School"
- board text added: "Oliver O"
- board text added: "another duck"
- board text added: "light thing"
- board text added: "orpheus"
- board text added: "pls dont steal this ty"
- board text added: "self-promotion"
- board text added: "this bag belongs to"
- board text added: "tree"
