File: solder.kicad_sch (KiCad schematic)
At the start: 6 parts, among them Q2 NPN

Commit message: PCB Draft 1
Parts:
- BT1: renamed from BT2; footprint (none) -> Battery:BatteryHolder_Keystone_3034_1x20mm
- D1: renamed from D2; footprint (none) -> LED_THT:LED_D5.0mm
- Q1: renamed from Q2; footprint (none) -> Package_TO_SOT_THT:TO-92L_HandSolder
- R1: renamed from R5; footprint (none) -> OptoDevice:R_LDR_5.1x4.3mm_P3.4mm_Vertical
- RV1, RV2: footprint (none) -> Potentiometer_THT:Potentiometer_Vishay_T73YP_Vertical
Changed lines of the file:
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@@
 			)
 		)
-		(property "Footprint" ""
+		(property "Footprint" "Potentiometer_THT:Potentiometer_Vishay_T73YP_Vertical"
 			(at 144.78 74.93 0)
 			(effects
@@
 		(dnp no)
 		(fields_autoplaced yes)
-		(property "Reference" "Q2"
+		(property "Reference" "Q1"
 			(at 149.86 100.3299 0)
 			(effects
@@
 			)
 		)
-		(property "Footprint" ""
+		(property "Footprint" "Package_TO_SOT_THT:TO-92L_HandSolder"
 			(at 208.28 101.6 0)
 			(effects
@@
 			(project ""
 				(path "/111f090e-f09b-4f8c-b614-bde9cc0cc8f4"
-					(reference "Q2")
+					(reference "Q1")
 					(unit 1)
 				)
@@
 		(dnp no)
 		(fields_autoplaced yes)
-		(property "Reference" "D2"
+		(property "Reference" "D1"
 			(at 149.86 86.0424 90)
 			(effects
@@
 			)
 		)
-		(property "Footprint" ""
+		(property "Footprint" "LED_THT:LED_D5.0mm"
 			(at 147.32 88.9 0)
 			(effects
@@
 			(project ""
 				(path "/111f090e-f09b-4f8c-b614-bde9cc0cc8f4"
-					(reference "D2")
+					(reference "D1")
 					(unit 1)
 				)
@@
 		(dnp no)
 		(fields_autoplaced yes)
-		(property "Reference" "R5"
+		(property "Reference" "R1"
 			(at 139.7 110.4899 0)
 			(effects
@@
 			)
 		)
-		(property "Footprint" ""
+		(property "Footprint" "OptoDevice:R_LDR_5.1x4.3mm_P3.4mm_Vertical"
 			(at 138.43 118.11 90)
 			(effects
@@
 			(project ""
 				(path "/111f090e-f09b-4f8c-b614-bde9cc0cc8f4"
-					(reference "R5")
+					(reference "R1")
 					(unit 1)
 				)
@@
 			)
 		)
-		(property "Footprint" ""
+		(property "Footprint" "Potentiometer_THT:Potentiometer_Vishay_T73YP_Vertical"
 			(at 133.35 82.55 0)
 			(effects
@@
 		(dnp no)
 		(fields_autoplaced yes)
-		(property "Reference" "BT2"
+		(property "Reference" "BT1"
 			(at 121.92 87.0584 0)
 			(effects
@@
 			)
 		)
-		(property "Footprint" ""
+		(property "Footprint" "Battery:BatteryHolder_Keystone_3034_1x20mm"
 			(at 118.11 88.646 90)
 			(effects
@@
 			(project ""
 				(path "/111f090e-f09b-4f8c-b614-bde9cc0cc8f4"
-					(reference "BT2")
-					(unit 1)
-				)
+					(reference "BT1")
+					(unit 1)
+				)
