File: solder.kicad_sch (KiCad schematic)
At the start: 6 parts, among them Q1 NPN

Commit message: add resistor
Parts:
- added R2: 5K1, Resistor_THT:R_Axial_DIN0207_L6.3mm_D2.5mm_P7.62mm_Horizontal, symbol Device:R
Connections:
- net at Q1.2 (B), R1.1: now also R2.2; no longer RV1.2
- new net: R2.1, RV1.2
Other:
- moved on the sheet: RV1
Changed lines of the file:
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@@
 	)
 	(junction
-		(at 118.11 83.82)
+		(at 118.11 77.47)
 		(diameter 0)
 		(color 0 0 0 0)
@@
 	)
 	(no_connect
-		(at 135.89 83.82)
+		(at 129.54 77.47)
 	)
 	(wire
@@
 	(wire
 		(pts
-			(xy 118.11 68.58) (xy 118.11 83.82)
+			(xy 118.11 68.58) (xy 118.11 77.47)
+		)
+		(stroke
+			(width 0)
+			(type default)
+		)
+	)
+	(wire
+		(pts
+			(xy 118.11 77.47) (xy 118.11 92.71)
 		)
 		(stroke
@@
 	(wire
 		(pts
+			(xy 132.08 76.2) (xy 130.81 76.2)
+		)
+		(stroke
+			(width 0)
+			(type default)
+		)
+	)
+	(wire
+		(pts
 			(xy 147.32 92.71) (xy 147.32 96.52)
 		)
@@
 	(wire
 		(pts
-			(xy 118.11 83.82) (xy 128.27 83.82)
-		)
-		(stroke
-			(width 0)
-			(type default)
-		)
-	)
-	(wire
-		(pts
-			(xy 118.11 92.71) (xy 118.11 83.82)
-		)
-		(stroke
-			(width 0)
-			(type default)
-		)
-	)
-	(wire
-		(pts
-			(xy 142.24 92.71) (xy 142.24 80.01)
+			(xy 130.81 73.66) (xy 125.73 73.66)
+		)
+		(stroke
+			(width 0)
+			(type default)
+		)
+	)
+	(wire
+		(pts
+			(xy 118.11 77.47) (xy 121.92 77.47)
+		)
+		(stroke
+			(width 0)
+			(type default)
+		)
+	)
+	(wire
+		(pts
+			(xy 142.24 92.71) (xy 142.24 76.2)
 		)
 		(stroke
@@
 	(wire
 		(pts
+			(xy 130.81 76.2) (xy 130.81 73.66)
+		)
+		(stroke
+			(width 0)
+			(type default)
+		)
+	)
+	(wire
+		(pts
 			(xy 137.16 92.71) (xy 142.24 92.71)
 		)
@@
 	(wire
 		(pts
-			(xy 142.24 80.01) (xy 132.08 80.01)
+			(xy 142.24 76.2) (xy 139.7 76.2)
 		)
 		(stroke
@@
 	)
 	(symbol
+		(lib_id "Device:R")
+		(at 135.89 76.2 90)
+		(unit 1)
+		(exclude_from_sim no)
+		(in_bom yes)
+		(on_board yes)
+		(dnp no)
+		(fields_autoplaced yes)
+		(property "Reference" "R2"
+			(at 135.89 69.85 90)
+			(effects
+				(font
+					(size 1.27 1.27)
+				)
+			)
+		)
+		(property "Value" "5K1"
+			(at 135.89 72.39 90)
+			(effects
+				(font
+					(size 1.27 1.27)
+				)
+			)
+		)
+		(property "Footprint" "Resistor_THT:R_Axial_DIN0207_L6.3mm_D2.5mm_P7.62mm_Horizontal"
+			(at 135.89 77.978 90)
+			(effects
+				(font
+					(size 1.27 1.27)
+				)
+				(hide yes)
+			)
+		)
+		(property "Datasheet" "~"
+			(at 135.89 76.2 0)
+			(effects
+				(font
+					(size 1.27 1.27)
+				)
+				(hide yes)
+			)
+		)
+		(property "Description" "Resistor"
+			(at 135.89 76.2 0)
+			(effects
+				(font
+					(size 1.27 1.27)
+				)
+				(hide yes)
+			)
+		)
+		(pin "2"
+		)
+		(pin "1"
+		)
+		(instances
+			(project ""
+				(path "/111f090e-f09b-4f8c-b614-bde9cc0cc8f4"
+					(reference "R2")
+					(unit 1)
+				)
+			)
+		)
+	)
+	(symbol
 		(lib_id "Device:R_Potentiometer")
-		(at 132.08 83.82 90)
+		(at 125.73 77.47 90)
 		(unit 1)
 		(exclude_from_sim no)
@@
 		(fields_autoplaced yes)
 		(property "Reference" "RV1"
-			(at 132.08 87.63 90)
+			(at 125.73 81.28 90)
 			(effects
 				(font
@@
 		)
 		(property "Value" "R_Potentiometer"
-			(at 132.08 90.17 90)
+			(at 125.73 83.82 90)
 			(effects
 				(font
@@
 		)
 		(property "Footprint" "Potentiometer_THT:Potentiometer_Vishay_T73YP_Vertical"
-			(at 132.08 83.82 0)
+			(at 125.73 77.47 0)
 			(effects
 				(font
@@
 		)
 		(property "Datasheet" "~"
-			(at 132.08 83.82 0)
+			(at 125.73 77.47 0)
 			(effects
 				(font
@@
 		)
 		(property "Description" "Potentiometer"
-			(at 132.08 83.82 0)
-			(effects
-				(font
+			(at 125.73 77.47 0)
+			(effects
+				(font

Commit message: update images and pcb
Parts:
- added R3: 5K1, Resistor_THT:R_Axial_DIN0207_L6.3mm_D2.5mm_P7.62mm_Horizontal, symbol Device:R
Connections:
- net at Q1.2 (B), R1.1: now also R3.1; no longer R2.2
- new net: R2.2, R3.2
Changed lines of the file:
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@@
+	(wire
+		(pts
+			(xy 139.7 76.2) (xy 142.24 76.2)
+		)
+		(stroke
+			(width 0)
+			(type default)
+		)
+	)
 	(wire
 		(pts
@@
 	(wire
 		(pts
+			(xy 142.24 87.63) (xy 142.24 92.71)
+		)
+		(stroke
+			(width 0)
+			(type default)
+		)
+	)
+	(wire
+		(pts
 			(xy 147.32 120.65) (xy 137.16 120.65)
 		)
@@
 	(wire
 		(pts
-			(xy 142.24 92.71) (xy 142.24 76.2)
+			(xy 142.24 76.2) (xy 142.24 80.01)
 		)
 		(stroke
@@
 		(pts
 			(xy 137.16 101.6) (xy 139.7 101.6)
-		)
-		(stroke
-			(width 0)
-			(type default)
-		)
-	)
-	(wire
-		(pts
-			(xy 142.24 76.2) (xy 139.7 76.2)
 		)
 		(stroke
@@
 					(unit 1)
 				)
+			)
+		)
+	)
+	(symbol
+		(lib_id "Device:R")
+		(at 142.24 83.82 180)
+		(unit 1)
+		(exclude_from_sim no)
+		(in_bom yes)
+		(on_board yes)
+		(dnp no)
+		(fields_autoplaced yes)
+		(property "Reference" "R3"
+			(at 144.78 82.5499 0)
+			(effects
+				(font
+					(size 1.27 1.27)
+				)
+				(justify right)
+			)
+		)
+		(property "Value" "5K1"
+			(at 144.78 85.0899 0)
+			(effects
+				(font
+					(size 1.27 1.27)
+				)
+				(justify right)
+			)
+		)
+		(property "Footprint" "Resistor_THT:R_Axial_DIN0207_L6.3mm_D2.5mm_P7.62mm_Horizontal"
+			(at 144.018 83.82 90)
+			(effects
+				(font
+					(size 1.27 1.27)
+				)
+				(hide yes)
+			)
+		)
+		(property "Datasheet" "~"
+			(at 142.24 83.82 0)
+			(effects
+				(font
+					(size 1.27 1.27)
+				)
+				(hide yes)
+			)
+		)
+		(property "Description" "Resistor"
+			(at 142.24 83.82 0)
+			(effects
+				(font
+					(size 1.27 1.27)
+				)
+				(hide yes)
+			)
+		)
+		(pin "2"
+		)
+		(pin "1"
+		)
+		(instances
+			(project "solder"
+				(path "/111f090e-f09b-4f8c-b614-bde9cc0cc8f4"
+					(reference "R3")
+					(unit 1)
+				)
